File: UnUn_BNC/UnUn_BNC.kicad_pcb (KiCad board)
At the start: 2 copper layers, 37.3 x 54.6 mm, 14 parts, among them J1 BNC, J3 B_THT_Pad, J4 B_SMD_PAD, J5 A_THT_Pad, J6 A_SMD_PAD, U2 Core

Commit message: fixed issue with netlist (no functional change, only to prevent DRC Error at Aisler.net)
Connections:
- U2 pad 4: Net-(U1-Pad1) -> Net-(C1-Pad1)
Changed lines of the file:
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@@
   (net 2 "GND")
   (net 3 "Net-(H1-Pad1)")
-  (net 4 "Net-(U1-Pad1)")
   (footprint "UniBalunLibrary:FT82_Balun" (layer "F.Cu")
     (at 117.602 65.532)
@@
       (net 2 "GND") (pinfunction "a") (pintype "input"))
     (pad "4" thru_hole roundrect (at -3.7 13.2) (size 2.55 2.55) (drill 1.55) (layers *.Cu *.Mask) (roundrect_rratio 0.09803882353)
-      (net 4 "Net-(U1-Pad1)") (pinfunction "b'") (pintype "output"))
+      (net 1 "Net-(C1-Pad1)") (pinfunction "b'") (pintype "output"))
     (pad "5" thru_hole roundrect (at 4.5212 -12.7) (size 2.55 2.55) (drill 1.55) (layers *.Cu *.Mask) (roundrect_rratio 0.09803882353)
       (net 3 "Net-(H1-Pad1)") (pinfunction "x") (pintype "output"))
@@
     (effects (font (size 1.5 1.5) (thickness 0.25)))
   )
+  (segment (start 113.932 79.068) (end 114.025 78.975) (width 1.3) (layer "F.Cu") (net 1))
   (segment (start 113.8 82.425) (end 112.595 82.425) (width 1.3) (layer "B.Cu") (net 1))
   (segment (start 117.075 82.425) (end 115.135 82.425) (width 1.3) (layer "B.Cu") (net 1))
@@
   (segment (start 113.8 82.425) (end 113.8 79.175) (width 1.3) (layer "B.Cu") (net 1))
   (segment (start 117.525 82.875) (end 117.075 82.425) (width 1.3) (layer "B.Cu") (net 1))
+  (segment (start 114.018 78.668) (end 113.925 78.575) (width 1.3) (layer "B.Cu") (net 1))
   (segment (start 115.135 82.425) (end 113.8 82.425) (width 1.3) (layer "B.Cu") (net 1))
   (segment (start 117.525 87.375) (end 117.525 82.875) (width 1.3) (layer "B.Cu") (net 1))
@@
   (segment (start 128.016 48.26) (end 132.08 52.324) (width 1.3) (layer "B.Cu") (net 3))
   (segment (start 125.5268 55.6768) (end 127 57.15) (width 1.3) (layer "B.Cu") (net 3))
-  (segment (start 113.932 79.068) (end 114.025 78.975) (width 1.3) (layer "F.Cu") (net 4))
-  (segment (start 114.018 78.668) (end 113.925 78.575) (width 1.3) (layer "B.Cu") (net 4))
   (zone (net 2) (net_name "GND") (layer "B.Cu") (hatch edge 0.508)
     (connect_pads yes (clearance 0.8))
